File: _autosave-Gigalux.kicad_pcb (KiCad board)
At the start: 2 copper layers, 101.6 x 17.8 mm, 9 parts, among them P1 IN, P2 OUT, U1 TLC5971

Commit message: Updates
Parts:
- U1: footprint Zetaohm:TLC59711 -> TLC59711
- turned D1 to 90 degrees
Routing:
- net SCKI: track 58.2 -> 0.15 mm, vias 8 -> 0
- net SDTI: track 47.8 -> 2.41 mm, vias 4 -> 2
- net +5V: track 187.9 -> 143.0 mm, vias 3 -> 2
- net (no net): track 0.00 -> 3.99 mm, vias 0 -> 3
- net B2: track 30.6 -> 28.3 mm, vias 5 -> 2
- net R1: track 20.8 -> 21.8 mm
- net G0: track 44.5 -> 45.4 mm, vias 3 -> 2
- net B1: track 26.1 -> 26.8 mm
- net R2: track 25.8 -> 25.5 mm, vias 3 -> 2
- net R0: vias 3 -> 2
- net G2: vias 4 -> 3
Other:
- net class +5V added: clearance 0.61, trace_width 5, via_dia 2.5, via_drill 1
- net class PWR added: clearance 0.61, trace_width 5, via_dia 0.6, via_drill 0.4
