File: Gigalux.sch (KiCad schematic (older format))
At the start: 7 parts, among them U1 TLC5971

Commit message: Daily Commit
Parts:
- gave numbers to parts that had none: 1
Changed lines of the file:
@@
 LIBS:contrib
 LIBS:valves
-LIBS:ZettaOhm
+LIBS:Zetaohm
 LIBS:Gigalux-cache
 EELAYER 25 0
@@
 $EndComp
 $Comp
-L +5V #PWR01
+L +5V #PWR1
 U 1 1 559B5889
 P 3950 1800
-F 0 "#PWR01" H 3950 1650 50  0001 C CNN
+F 0 "#PWR1" H 3950 1650 50  0001 C CNN
 F 1 "+5V" H 3950 1940 50  0000 C CNN
 F 2 "" H 3950 1800 60  0000 C CNN
@@
 $EndComp
 $Comp
-L +5V #PWR02
+L +5V #PWR3
 U 1 1 559B5911
 P 7100 3050
-F 0 "#PWR02" H 7100 2900 50  0001 C CNN
+F 0 "#PWR3" H 7100 2900 50  0001 C CNN
 F 1 "+5V" H 7100 3190 50  0000 C CNN
 F 2 "" H 7100 3050 60  0000 C CNN
@@
 $EndComp
 $Comp
-L GND #PWR04
+L GND #PWR4
 U 1 1 559B6F8D
 P 4250 3600
-F 0 "#PWR04" H 4250 3350 50  0001 C CNN
+F 0 "#PWR4" H 4250 3350 50  0001 C CNN
 F 1 "GND" H 4250 3450 50  0000 C CNN
 F 2 "" H 4250 3600 60  0000 C CNN
@@
 	3250 2500 2850 2500
 $Comp
-L +5V #PWR05
+L +5V #PWR2
 U 1 1 559B811D
 P 9250 1800
-F 0 "#PWR05" H 9250 1650 50  0001 C CNN
+F 0 "#PWR2" H 9250 1650 50  0001 C CNN
 F 1 "+5V" H 9250 1940 50  0000 C CNN
 F 2 "" H 9250 1800 60  0000 C CNN
@@
 	8550 2500 8150 2500
 $Comp
-L +5V #PWR07
+L +5V #PWR6
 U 1 1 559B81CB
 P 3950 5050
-F 0 "#PWR07" H 3950 4900 50  0001 C CNN
+F 0 "#PWR6" H 3950 4900 50  0001 C CNN
 F 1 "+5V" H 3950 5190 50  0000 C CNN
 F 2 "" H 3950 5050 60  0000 C CNN
@@
 	3250 5750 2850 5750
 $Comp
-L +5V #PWR09
+L +5V #PWR7
 U 1 1 559B81ED
 P 9250 5050
-F 0 "#PWR09" H 9250 4900 50  0001 C CNN
+F 0 "#PWR7" H 9250 4900 50  0001 C CNN
 F 1 "+5V" H 9250 5190 50  0000 C CNN
 F 2 "" H 9250 5050 60  0000 C CNN
@@
 Connection ~ 4750 3500
 $Comp
-L C C?
+L C C1
 U 1 1 559C354A
 P 8000 3550
-F 0 "C?" H 8025 3650 50  0000 L CNN
+F 0 "C1" H 8025 3650 50  0000 L CNN
 F 1 "C" H 8025 3450 50  0000 L CNN
 F 2 "Capacitors_SMD:C_0805_HandSoldering" H 8038 3400 30  0001 C CNN
@@
 	8000 3300 8000 3400
 $Comp
-L GND #PWR?
+L GND #PWR5
 U 1 1 559C478E
 P 8000 3800
-F 0 "#PWR?" H 8000 3550 50  0001 C CNN
+F 0 "#PWR5" H 8000 3550 50  0001 C CNN
 F 1 "GND" H 8000 3650 50  0000 C CNN
 F 2 "" H 8000 3800 60  0000 C CNN

Commit message: Updates
Parts:
- added P1, P2: CONN_01X04, Pin_Headers:Pin_Header_Straight_1x04, symbol CONN_01X04
- D1, D2, D3, D4: footprint (none) -> Zetaohm:AAAF5051-04
- R1: footprint (none) -> Capacitors_SMD:C_0805_HandSoldering
- U1: footprint (none) -> Zetaohm:TLC59711
Connections:
- net +5V: now also P1.4 (P4), P2.4 (P4)
- net GND: now also P1.1 (P1), P2.1 (P1)
- net SCKO: now also P2.2 (P2); no longer U1.10 (SCKI)
- net SDTI: now also P1.3 (P3)
- net SDTO: now also P2.3 (P3)
- new net SCKI: P1.2 (P2), U1.10 (SCKI)
Changed lines of the file:
@@
 F 0 "U1" H 6300 4450 60  0000 C CNN
 F 1 "TLC5971" H 5900 4450 60  0000 C CNN
-F 2 "" H 6250 4000 60  0001 C CNN
+F 2 "Zetaohm:TLC59711" H 6250 4000 60  0001 C CNN
 F 3 "" H 6250 4000 60  0000 C CNN
 	1    6050 4000
@@
 $EndComp
 $Comp
-L +5V #PWR1
+L +5V #PWR01
 U 1 1 559B5889
 P 3950 1800
-F 0 "#PWR1" H 3950 1650 50  0001 C CNN
+F 0 "#PWR01" H 3950 1650 50  0001 C CNN
 F 1 "+5V" H 3950 1940 50  0000 C CNN
 F 2 "" H 3950 1800 60  0000 C CNN
@@
 $EndComp
 $Comp
-L +5V #PWR3
+L +5V #PWR02
 U 1 1 559B5911
 P 7100 3050
-F 0 "#PWR3" H 7100 2900 50  0001 C CNN
+F 0 "#PWR02" H 7100 2900 50  0001 C CNN
 F 1 "+5V" H 7100 3190 50  0000 C CNN
 F 2 "" H 7100 3050 60  0000 C CNN
@@
 F 0 "D1" H 3450 2650 50  0000 C CNN
 F 1 "AAAF5051-04" H 3450 1950 50  0000 C CNN
-F 2 "" H 3405 2250 50  0001 C CNN
+F 2 "Zetaohm:AAAF5051-04" H 3405 2250 50  0001 C CNN
 F 3 "" H 3405 2250 50  0000 C CNN
 	1    3450 2300
@@
 $EndComp
 $Comp
-L GND #PWR4
+L GND #PWR03
 U 1 1 559B6F8D
 P 4250 3600
-F 0 "#PWR4" H 4250 3350 50  0001 C CNN
+F 0 "#PWR03" H 4250 3350 50  0001 C CNN
 F 1 "GND" H 4250 3450 50  0000 C CNN
 F 2 "" H 4250 3600 60  0000 C CNN
@@
 F 0 "R1" V 5050 3600 50  0000 C CNN
 F 1 "Resistor" V 4990 3490 50  0001 C CNN
-F 2 "" V 5030 3500 30  0001 C CNN
+F 2 "Capacitors_SMD:C_0805_HandSoldering" V 5030 3500 30  0001 C CNN
 F 3 "" H 5100 3490 30  0000 C CNN
 	1    5100 3500
@@
 	7100 3750 6600 3750
 Wire Wire Line
-	7100 3050 7100 3750
+	7100 3050 7100 3300
+Wire Wire Line
+	7100 3300 7100 3750
 Wire Wire Line
 	4250 3600 4250 3500
 Wire Wire Line
-	4250 3500 5000 3500
+	4250 3500 4750 3500
+Wire Wire Line
+	4750 3500 5000 3500
 Wire Wire Line
 	4750 3750 5500 3750
@@
 	4950 4450 5500 4450
 Text GLabel 4650 4550 0    60   Output ~ 0
-SCKO
+SCKI
 Wire Wire Line
 	4650 4550 5500 4550
@@
 	3250 2500 2850 2500
 $Comp
-L +5V #PWR2
+L +5V #PWR04
 U 1 1 559B811D
 P 9250 1800
-F 0 "#PWR2" H 9250 1650 50  0001 C CNN
+F 0 "#PWR04" H 9250 1650 50  0001 C CNN
 F 1 "+5V" H 9250 1940 50  0000 C CNN
 F 2 "" H 9250 1800 60  0000 C CNN
@@
 F 0 "D2" H 8750 2650 50  0000 C CNN
 F 1 "AAAF5051-04" H 8750 1950 50  0000 C CNN
-F 2 "" H 8705 2250 50  0001 C CNN
+F 2 "Zetaohm:AAAF5051-04" H 8705 2250 50  0001 C CNN
 F 3 "" H 8705 2250 50  0000 C CNN
 	1    8750 2300
@@
 	8550 2500 8150 2500
 $Comp
-L +5V #PWR6
+L +5V #PWR05
 U 1 1 559B81CB
 P 3950 5050
-F 0 "#PWR6" H 3950 4900 50  0001 C CNN
+F 0 "#PWR05" H 3950 4900 50  0001 C CNN
 F 1 "+5V" H 3950 5190 50  0000 C CNN
 F 2 "" H 3950 5050 60  0000 C CNN
@@
 F 0 "D3" H 3450 5900 50  0000 C CNN
 F 1 "AAAF5051-04" H 3450 5200 50  0000 C CNN
-F 2 "" H 3405 5500 50  0001 C CNN
+F 2 "Zetaohm:AAAF5051-04" H 3405 5500 50  0001 C CNN
 F 3 "" H 3405 5500 50  0000 C CNN
 	1    3450 5550
@@
 	3250 5750 2850 5750
 $Comp
-L +5V #PWR7
+L +5V #PWR06
 U 1 1 559B81ED
 P 9250 5050
-F 0 "#PWR7" H 9250 4900 50  0001 C CNN
+F 0 "#PWR06" H 9250 4900 50  0001 C CNN
 F 1 "+5V" H 9250 5190 50  0000 C CNN
 F 2 "" H 9250 5050 60  0000 C CNN
@@
 F 0 "D4" H 8750 5900 50  0000 C CNN
 F 1 "AAAF5051-04" H 8750 5200 50  0000 C CNN
-F 2 "" H 8705 5500 50  0001 C CNN
+F 2 "Zetaohm:AAAF5051-04" H 8705 5500 50  0001 C CNN
 F 3 "" H 8705 5500 50  0000 C CNN
 	1    8750 5550
@@
 $EndComp
 Wire Wire Line
-	6800 3300 8000 3300
+	6800 3300 7100 3300
+Wire Wire Line
+	7100 3300 8000 3300
 Wire Wire Line
 	8000 3300 8000 3400
 $Comp
-L GND #PWR5
+L GND #PWR07
 U 1 1 559C478E
 P 8000 3800
-F 0 "#PWR5" H 8000 3550 50  0001 C CNN
+F 0 "#PWR07" H 8000 3550 50  0001 C CNN
 F 1 "GND" H 8000 3650 50  0000 C CNN
 F 2 "" H 8000 3800 60  0000 C CNN
@@
 Wire Wire Line
 	6800 3650 6800 3300
+$Comp
+L CONN_01X04 P2
+U 1 1 559ED7D7
+P 6350 1400
+F 0 "P2" H 6350 1650 50  0000 C CNN
+F 1 "CONN_01X04" V 6450 1400 50  0000 C CNN
+F 2 "Pin_Headers:Pin_Header_Straight_1x04" H 6350 1400 60  0001 C CNN
+F 3 "" H 6350 1400 60  0000 C CNN
+	1    6350 1400
+	-1   0    0    1
+$EndComp
+Text GLabel 5000 1450 2    60   Output ~ 0
+SCKI
+Text GLabel 5350 1350 2    60   Output ~ 0
+SDTI
+Text GLabel 7200 1350 2    60   Output ~ 0
+SDTO
+Text GLabel 6850 1450 2    60   Output ~ 0
+SCKO
+$Comp
+L GND #PWR08
+U 1 1 559EE260
+P 6950 1750
+F 0 "#PWR08" H 6950 1500 50  0001 C CNN
+F 1 "GND" H 6950 1600 50  0000 C CNN
+F 2 "" H 6950 1750 60  0000 C CNN
+F 3 "" H 6950 1750 60  0000 C CNN
+	1    6950 1750
+	1    0    0    -1
+$EndComp
+Wire Wire Line
+	6550 1550 6950 1550
+Wire Wire Line
+	6950 1550 6950 1750
+Wire Wire Line
+	6550 1450 6850 1450
+$Comp
+L +5V #PWR09
+U 1 1 559EE378
+P 6950 1050
+F 0 "#PWR09" H 6950 900 50  0001 C CNN
+F 1 "+5V" H 6950 1190 50  0000 C CNN
+F 2 "" H 6950 1050 60  0000 C CNN
+F 3 "" H 6950 1050 60  0000 C CNN
+	1    6950 1050
+	1    0    0    -1
+$EndComp
+$Comp
+L CONN_01X04 P1
+U 1 1 559EEDE5
+P 4500 1400
+F 0 "P1" H 4500 1650 50  0000 C CNN
+F 1 "CONN_01X04" V 4600 1400 50  0000 C CNN
+F 2 "Pin_Headers:Pin_Header_Straight_1x04" H 4500 1400 60  0001 C CNN
+F 3 "" H 4500 1400 60  0000 C CNN
+	1    4500 1400
+	-1   0    0    1
+$EndComp
+$Comp
+L GND #PWR010
+U 1 1 559EEDED
+P 5100 1750
+F 0 "#PWR010" H 5100 1500 50  0001 C CNN
+F 1 "GND" H 5100 1600 50  0000 C CNN
+F 2 "" H 5100 1750 60  0000 C CNN
+F 3 "" H 5100 1750 60  0000 C CNN
+	1    5100 1750
+	1    0    0    -1
+$EndComp
+Wire Wire Line
+	4700 1550 5100 1550
+Wire Wire Line
+	5100 1550 5100 1750
+Wire Wire Line
+	4700 1450 5000 1450
+Wire Wire Line
+	4700 1350 5350 1350
+$Comp
+L +5V #PWR011
+U 1 1 559EEDF7
+P 5100 1050
+F 0 "#PWR011" H 5100 900 50  0001 C CNN
+F 1 "+5V" H 5100 1190 50  0000 C CNN
+F 2 "" H 5100 1050 60  0000 C CNN
+F 3 "" H 5100 1050 60  0000 C CNN
+	1    5100 1050
+	1    0    0    -1
+$EndComp
+Wire Wire Line
+	6550 1350 7200 1350
+Wire Wire Line
+	4700 1250 5100 1250
+Wire Wire Line
+	5100 1250 5100 1050
+Wire Wire Line
+	6550 1250 6950 1250
+Wire Wire Line
+	6950 1250 6950 1050
 $EndSCHEMATC

Commit message: Fixed pinouts for TLC5711, fixed board layout.
This is the one that was sent to OSH park on 7/15
Parts:
- P1, P2: footprint Pin_Headers:Pin_Header_Straight_1x04 -> Zetaohm:KK396-4Pin
Changed lines of the file:
@@
 	7100 3750 6600 3750
 Wire Wire Line
-	7100 3050 7100 3300
-Wire Wire Line
-	7100 3300 7100 3750
+	7100 3050 7100 3750
 Wire Wire Line
 	4250 3600 4250 3500
 Wire Wire Line
-	4250 3500 4750 3500
-Wire Wire Line
-	4750 3500 5000 3500
+	4250 3500 5000 3500
 Wire Wire Line
 	4750 3750 5500 3750
@@
 $EndComp
 Wire Wire Line
-	6800 3300 7100 3300
-Wire Wire Line
-	7100 3300 8000 3300
+	6800 3300 8000 3300
 Wire Wire Line
 	8000 3300 8000 3400
@@
 F 0 "P2" H 6350 1650 50  0000 C CNN
 F 1 "CONN_01X04" V 6450 1400 50  0000 C CNN
-F 2 "Pin_Headers:Pin_Header_Straight_1x04" H 6350 1400 60  0001 C CNN
+F 2 "Zetaohm:KK396-4Pin" H 6350 1400 60  0001 C CNN
 F 3 "" H 6350 1400 60  0000 C CNN
 	1    6350 1400
@@
 F 0 "P1" H 4500 1650 50  0000 C CNN
 F 1 "CONN_01X04" V 4600 1400 50  0000 C CNN
-F 2 "Pin_Headers:Pin_Header_Straight_1x04" H 4500 1400 60  0001 C CNN
+F 2 "Zetaohm:KK396-4Pin" H 4500 1400 60  0001 C CNN
 F 3 "" H 4500 1400 60  0000 C CNN
 	1    4500 1400
